Commit message: Update obj.xacro

File: src/heads/urdf/obj.xacro (robot description, xacro)
@@ -8,10 +8,10 @@
     <collision name='collision'>
       <geometry>
-	    <box size="1 1 0.5"/>
+	    <box size="0.2 1 1.5"/>
       </geometry>
     </collision>
     <visual name='visual'>
       <geometry>
-	    <box size="1 1 0.5"/>
+	    <box size="0.2 1 1.5"/>
       </geometry>
       <material name="black"/>
@@ -19,5 +19,5 @@
     <inertial>
       <origin xyz="0 0 0" />
-      <mass value="10.0" />
+      <mass value="50.0" />
       <inertia  ixx="1.0" ixy="0.0"  ixz="0.0"  iyy="100.0"  iyz="0.0"  izz="1.0" />
     </inertial>
@@ -30,5 +30,5 @@
   <joint name="camera_joint" type="fixed">
     <axis xyz="0 1 0" />
-    <origin xyz="${camera_size} 0 0.5" rpy="0 0 0"/>
+    <origin xyz="${camera_size} 0 0.85" rpy="0 0 0"/>
     <parent link="table_link"/>
     <child link="camera_link"/>
