Commit message: Pridetas stl galvos modelis

File: src/heads/urdf/head.xacro (robot description, xacro)
@@ -9,13 +9,42 @@
   <xacro:include filename="$(find heads)/urdf/head.gazebo" />
   <link name="world"/>
+  <link name="torse_link">
+    <collision name='collision'>
+      <geometry>
+	    <box size="0.5 0.5 1.6"/>
+      </geometry>
+    </collision>
+    <visual name='visual'>
+      <geometry>
+	    <box size="0.5 0.5 1.6"/>
+      </geometry>
+      <material name="black"/>
+    </visual>
+    <inertial>
+      <origin xyz="0 0 0" />
+      <mass value="70.0" />
+      <inertia  ixx="1.0" ixy="0.0"  ixz="0.0"  iyy="100.0"  iyz="0.0"  izz="1.0" />
+    </inertial>
+  </link>
+  <joint name="torse_joint" type="floating">
+    <origin xyz="0 0 0.8" rpy="0 0 0"/>
+    <parent link="world"/>
+    <child link="torse_link"/>
+  </joint>
   <link name="base_link">
     <collision>
       <geometry>
-	    <mesh filename="file:///home/deivydas/Desktop/bolvanka/bolvanka.obj"/>
+	    <mesh filename="file:////home/deivydas/Desktop/face.stl"/>
+     <!-- <uri>package://heads/models/face.stl</uri>
+      <scale>0.001 0.001 0.001</scale>
+    -->
       </geometry>
     </collision>
     <visual>
       <geometry>
-	    <mesh filename="file:///home/deivydas/Desktop/bolvanka/bolvanka.obj"/>
+	    <mesh filename="file:////home/deivydas/Desktop/face.stl"/>
+     <!-- <uri>package://heads/models/face.stl</uri>
+      <scale>0.001 0.001 0.001</scale>
+    -->
       </geometry>
       <material name="orange"/>
@@ -27,6 +56,7 @@
     </inertial>
   </link>
-  <joint name="base_joint" type="floating">
-    <parent link="world"/>
+  <joint name="base_joint" type="fixed">
+    <origin xyz="0 0 0.9" rpy="0 0 0"/>
+    <parent link="torse_link"/>
     <child link="base_link"/>
   </joint>
@@ -67,13 +97,13 @@
     </inertial>
   </link>
-  <joint name="right_eye_joint" type="fixed">
+  <joint name="right_eye_joint" type="floating">
     <axis xyz="0 1 0" />
-    <origin xyz="${rad} ${rad} ${rad}" rpy="0 0 0"/>
+    <origin xyz="${rad} ${rad} ${rad}" rpy="0 0 1.57"/>
     <parent link="base_link"/>
     <child link="right_eye_link"/>
   </joint>
-  <joint name="left_eye_joint" type="fixed">
+  <joint name="left_eye_joint" type="floating">
     <axis xyz="0 1 0" />
-    <origin xyz="-${rad} ${rad} ${rad}" rpy="0 0 0"/>
+    <origin xyz="-${rad} ${rad} ${rad}" rpy="0 0 1.57"/>
     <parent link="base_link"/>
     <child link="left_eye_link"/>

Commit message: Continues joints to revolute

File: src/heads/urdf/head.xacro (robot description, xacro)
@@ -12,10 +12,10 @@
     <collision name='collision'>
       <geometry>
-	    <box size="0.5 0.5 1.6"/>
+        <mesh filename="package://heads/models/torso.dae"/>
       </geometry>
     </collision>
     <visual name='visual'>
       <geometry>
-	    <box size="0.5 0.5 1.6"/>
+        <mesh filename="package://heads/models/torso.dae"/>
       </geometry>
       <material name="black"/>
@@ -27,24 +27,47 @@
     </inertial>
   </link>
-  <joint name="torse_joint" type="floating">
-    <origin xyz="0 0 0.8" rpy="0 0 0"/>
+  <joint name="torse_joint" type="fixed">
+    <origin xyz="0 0 0.0" rpy="1.57 0 0"/>
     <parent link="world"/>
     <child link="torse_link"/>
   </joint>
-  <link name="base_link">
-    <collision>
-      <geometry>
-	    <mesh filename="file:////home/deivydas/Desktop/face.stl"/>
-     <!-- <uri>package://heads/models/face.stl</uri>
-      <scale>0.001 0.001 0.001</scale>
-    -->
-      </geometry>
-    </collision>
-    <visual>
-      <geometry>
-	    <mesh filename="file:////home/deivydas/Desktop/face.stl"/>
-     <!-- <uri>package://heads/models/face.stl</uri>
-      <scale>0.001 0.001 0.001</scale>
-    -->
+  <link name="head_yaw_link">
+    <inertial>
+      <origin xyz="0.137802209307 0.090396 0.0227196811405" rpy="0 0 0"/>
+      <mass value="0.10"/>
+      <inertia ixx="0.0" ixy="0.0" ixz="0.0" iyy="0.0" iyz="0.0" izz="0.0"/>
+    </inertial>
+  </link>
+  <joint name="head_yaw_joint" type="revolute">
+    <origin xyz="0 1.5 0.0" rpy="0 0 0"/>
+    <axis xyz="0 1 0"/>
+    <limit effort="1000.0" lower="-0.50" upper="0.5" velocity="0.5"/>
+    <parent link="torse_link"/>
+    <child link="head_yaw_link"/>
+  </joint>
+  <link name="head_pitch_link">
+    <inertial>
+      <origin xyz="0.137802209307 0.090396 0.0227196811405" rpy="0 0 0"/>
+      <mass value="0.10"/>
+      <inertia ixx="0.0" ixy="0.0" ixz="0.0" iyy="0.0" iyz="0.0" izz="0.0"/>
+    </inertial>
+  </link>
+  <joint name="head_pitch_joint" type="revolute">
+    <axis xyz="1 0 0"/>
+    <limit effort="1000.0" lower="-0.50" upper="0.5" velocity="0.5"/>
+    <parent link="head_yaw_link"/>
+    <child link="head_pitch_link"/>
+  </joint>
+  <link name="head_roll_link">
+    <collision>
+     <origin xyz="0 -1.5 0" rpy="0 0 0" />
+      <geometry>
+        <mesh filename="package://heads/models/head.dae"/>
+      </geometry>
+    </collision>
+    <visual>
+     <origin xyz="0 -1.5 0" rpy="0 0 0" />
+      <geometry>
+        <mesh filename="package://heads/models/head.dae"/>
       </geometry>
       <material name="orange"/>
@@ -52,14 +75,15 @@
     <inertial>
       <origin xyz="0 0 0.1" />
-      <mass value="1.0" />
-      <inertia  ixx="1.0" ixy="0.0"  ixz="0.0"  iyy="100.0"  iyz="0.0"  izz="1.0" />
-    </inertial>
-  </link>
-  <joint name="base_joint" type="fixed">
-    <origin xyz="0 0 0.9" rpy="0 0 0"/>
-    <parent link="torse_link"/>
-    <child link="base_link"/>
-  </joint>
-  <link name="left_eye_link">
+      <mass value="0.010" />
+      <inertia  ixx="1.0" ixy="0.0"  ixz="0.0"  iyy="100.0"  iyz="0.0"  izz="1.0" />
+    </inertial>
+  </link>
+  <joint name="head_roll_joint" type="revolute">
+    <axis xyz="0 0 1"/>
+    <limit effort="1000.0" lower="-0.50" upper="0.5" velocity="0.5"/>
+    <parent link="head_pitch_link"/>
+    <child link="head_roll_link"/>
+  </joint>
+<link name="left_eye_link">
     <collision>
       <geometry>
@@ -79,4 +103,35 @@
     </inertial>
   </link>
+  <joint name="left_eye_joint" type="fixed">
+    <origin xyz="${rad} ${rad} ${rad}" rpy="0 0 0"/>
+    <parent link="head_roll_link"/>
+    <child link="left_eye_link"/>
+  </joint>
+  <link name="left_eye_yaw_link">
+    <inertial>
+      <origin xyz="0.137802209307 0.090396 0.0227196811405" rpy="0 0 0"/>
+      <mass value="0.10"/>
+      <inertia ixx="0.0" ixy="0.0" ixz="0.0" iyy="0.0" iyz="0.0" izz="0.0"/>
+    </inertial>
+  </link>
+  <joint name="left_eye_yaw_joint" type="revolute">
+    <axis xyz="0 1 0"/>
+    <limit effort="1000.0" lower="-0.50" upper="0.5" velocity="0.5"/>
+    <parent link="left_eye_link"/>
+    <child link="left_eye_yaw_link"/>
+  </joint>
+  <link name="left_eye_pitch_link">
+    <inertial>
+      <origin xyz="0.137802209307 0.090396 0.0227196811405" rpy="0 0 0"/>
+      <mass value="0.10"/>
+      <inertia ixx="0.0" ixy="0.0" ixz="0.0" iyy="0.0" iyz="0.0" izz="0.0"/>
+    </inertial>
+  </link>
+  <joint name="left_eye_pitch_joint" type="revolute">
+    <axis xyz="1 0 0"/>
+    <limit effort="1000.0" lower="-0.50" upper="0.5" velocity="0.5"/>
+    <parent link="left_eye_yaw_link"/>
+    <child link="left_eye_pitch_link"/>
+  </joint>
   <link name="right_eye_link">
     <collision>
@@ -97,15 +152,34 @@
     </inertial>
   </link>
-  <joint name="right_eye_joint" type="floating">
-    <axis xyz="0 1 0" />
-    <origin xyz="${rad} ${rad} ${rad}" rpy="0 0 1.57"/>
-    <parent link="base_link"/>
+  <joint name="right_eye_joint" type="fixed">
+    <origin xyz="-${rad} ${rad} ${rad}" rpy="0 0 0"/>
+    <parent link="head_roll_link"/>
     <child link="right_eye_link"/>
   </joint>
-  <joint name="left_eye_joint" type="floating">
-    <axis xyz="0 1 0" />
-    <origin xyz="-${rad} ${rad} ${rad}" rpy="0 0 1.57"/>
-    <parent link="base_link"/>
-    <child link="left_eye_link"/>
+  <link name="right_eye_yaw_link">
+    <inertial>
+      <origin xyz="0.137802209307 0.090396 0.0227196811405" rpy="0 0 0"/>
+      <mass value="0.10"/>
+      <inertia ixx="0.0" ixy="0.0" ixz="0.0" iyy="0.0" iyz="0.0" izz="0.0"/>
+    </inertial>
+  </link>
+  <joint name="right_eye_yaw_joint" type="revolute">
+    <axis xyz="0 1 0"/>
+    <limit effort="1000.0" lower="-0.50" upper="0.5" velocity="0.5"/>
+    <parent link="right_eye_link"/>
+    <child link="right_eye_yaw_link"/>
+  </joint>
+  <link name="right_eye_pitch_link">
+    <inertial>
+      <origin xyz="0.137802209307 0.090396 0.0227196811405" rpy="0 0 0"/>
+      <mass value="0.10"/>
+      <inertia ixx="0.0" ixy="0.0" ixz="0.0" iyy="0.0" iyz="0.0" izz="0.0"/>
+    </inertial>
+  </link>
+  <joint name="right_eye_pitch_joint" type="revolute">
+    <axis xyz="1 0 0"/>
+    <limit effort="1000.0" lower="-0.50" upper="0.5" velocity="0.5"/>
+    <parent link="right_eye_yaw_link"/>
+    <child link="right_eye_pitch_link"/>
   </joint>
   <link name="left_camera_link">
@@ -146,14 +220,82 @@
   </link>
   <joint name="right_camera_joint" type="fixed">
-    <axis xyz="0 1 0" />
-    <origin xyz="0 0 0" rpy="0 0 0"/>
-    <parent link="right_eye_link"/>
+    <origin xyz="0 0 0" rpy="1.57 1.57 -3.14"/>
+    <parent link="right_eye_pitch_link"/>
     <child link="right_camera_link"/>
   </joint>
   <joint name="left_camera_joint" type="fixed">
-    <axis xyz="0 1 0" />
-    <origin xyz="0 0 0" rpy="0 0 0"/>
-    <parent link="left_eye_link"/>
+    <origin xyz="0 0 0" rpy="1.57 1.57 -3.14"/>
+    <parent link="left_eye_pitch_link"/>
     <child link="left_camera_link"/>
   </joint>
+  <transmission name="head_yaw_joint_tran">
+    <type>transmission_interface/SimpleTransmission</type>
+    <joint name="head_yaw_joint">
+      <hardwareInterface>hardware_interface/PositionJointInterface</hardwareInterface>
+    </joint>
+    <actuator name="head_yaw_joint_motor">
+      <hardwareInterface>hardware_interface/PositionJointInterface</hardwareInterface>
+      <mechanicalReduction>1</mechanicalReduction>
+    </actuator>
+  </transmission>
+  <transmission name="head_pitch_joint_tran">
+    <type>transmission_interface/SimpleTransmission</type>
+    <joint name="head_pitch_joint">
+      <hardwareInterface>hardware_interface/PositionJointInterface</hardwareInterface>
+    </joint>
+    <actuator name="head_pitch_joint_motor">
+      <hardwareInterface>hardware_interface/PositionJointInterface</hardwareInterface>
+      <mechanicalReduction>1</mechanicalReduction>
+    </actuator>
+  </transmission>
+  <transmission name="head_roll_joint_tran">
+    <type>transmission_interface/SimpleTransmission</type>
+    <joint name="head_roll_joint">
+      <hardwareInterface>hardware_interface/PositionJointInterface</hardwareInterface>
+    </joint>
+    <actuator name="head_roll_joint_motor">
+      <hardwareInterface>hardware_interface/PositionJointInterface</hardwareInterface>
+      <mechanicalReduction>1</mechanicalReduction>
+    </actuator>
+  </transmission>
+  <transmission name="left_eye_yaw_joint_tran">
+    <type>transmission_interface/SimpleTransmission</type>
+    <joint name="left_eye_yaw_joint">
+      <hardwareInterface>hardware_interface/PositionJointInterface</hardwareInterface>
+    </joint>
+    <actuator name="left_eye_yaw_joint_motor">
+      <hardwareInterface>hardware_interface/PositionJointInterface</hardwareInterface>
+      <mechanicalReduction>1</mechanicalReduction>
+    </actuator>
+  </transmission>
+  <transmission name="left_eye_pitch_joint_tran">
+    <type>transmission_interface/SimpleTransmission</type>
+    <joint name="left_eye_pitch_joint">
+      <hardwareInterface>hardware_interface/PositionJointInterface</hardwareInterface>
+    </joint>
+    <actuator name="left_eye_pitch_joint_motor">
+      <hardwareInterface>hardware_interface/PositionJointInterface</hardwareInterface>
+      <mechanicalReduction>1</mechanicalReduction>
+    </actuator>
+  </transmission>
+  <transmission name="right_eye_yaw_joint_tran">
+    <type>transmission_interface/SimpleTransmission</type>
+    <joint name="right_eye_yaw_joint">
+      <hardwareInterface>hardware_interface/PositionJointInterface</hardwareInterface>
+    </joint>
+    <actuator name="right_eye_yaw_joint_motor">
+      <hardwareInterface>hardware_interface/PositionJointInterface</hardwareInterface>
+      <mechanicalReduction>1</mechanicalReduction>
+    </actuator>
+  </transmission>
+  <transmission name="right_eye_pitch_joint_tran">
+    <type>transmission_interface/SimpleTransmission</type>
+    <joint name="right_eye_pitch_joint">
+      <hardwareInterface>hardware_interface/PositionJointInterface</hardwareInterface>
+    </joint>
+    <actuator name="right_eye_pitch_joint">
+      <hardwareInterface>hardware_interface/PositionJointInterface</hardwareInterface>
+      <mechanicalReduction>1</mechanicalReduction>
+    </actuator>
+  </transmission>
 </robot>

Commit message: Update head.xacro

File: src/heads/urdf/head.xacro (robot description, xacro)
@@ -4,5 +4,8 @@
   <xacro:property name="height1" value="2" />
   <xacro:property name="mass" value="5" />
-  <xacro:property name="rad" value="0.1" />
+  <xacro:property name="rad" value="0.05" />
+  <xacro:property name="rad_y" value="0.05" />
+  <xacro:property name="rad_z" value="0.08" />
+  <xacro:property name="rad_x" value="0.03" />
   <xacro:property name="rad_small" value="0.01" />
   <xacro:include filename="$(find heads)/urdf/materials.xacro" />
@@ -104,5 +107,5 @@
   </link>
   <joint name="left_eye_joint" type="fixed">
-    <origin xyz="${rad} ${rad} ${rad}" rpy="0 0 0"/>
+    <origin xyz="${rad_x} ${rad_y} ${rad_z}" rpy="0 0 0"/>
     <parent link="head_roll_link"/>
     <child link="left_eye_link"/>
@@ -153,5 +156,5 @@
   </link>
   <joint name="right_eye_joint" type="fixed">
-    <origin xyz="-${rad} ${rad} ${rad}" rpy="0 0 0"/>
+    <origin xyz="-${rad_x} ${rad_y} ${rad_z}" rpy="0 0 0"/>
     <parent link="head_roll_link"/>
     <child link="right_eye_link"/>
@@ -220,13 +223,49 @@
   </link>
   <joint name="right_camera_joint" type="fixed">
-    <origin xyz="0 0 0" rpy="1.57 1.57 -3.14"/>
+    <origin xyz="0 0 0" rpy="1.57 -1.57 -3.14"/>
     <parent link="right_eye_pitch_link"/>
     <child link="right_camera_link"/>
   </joint>
   <joint name="left_camera_joint" type="fixed">
-    <origin xyz="0 0 0" rpy="1.57 1.57 -3.14"/>
+    <origin xyz="0 0 0" rpy="1.57 -1.57 -3.14"/>
     <parent link="left_eye_pitch_link"/>
     <child link="left_camera_link"/>
   </joint>
+  <link name="left_sig_link">
+    <inertial>
+      <origin xyz="0 0 0" rpy="0 0 0"/>
+      <mass value="0.010"/>
+      <inertia ixx="0.0" ixy="0.0" ixz="0.0" iyy="0.0" iyz="0.0" izz="0.0"/>
+    </inertial>
+    <visual name='visual'>
+      <geometry>
+	    <box size="1 0.01 0.01"/>
+      </geometry>
+      <material name="black"/>
+    </visual>
+  </link>
+  <joint name="left_sig_joint" type="fixed">
+    <origin xyz="0.5 0 0" rpy="0 0 0"/>
+    <parent link="left_camera_link"/>
+    <child link="left_sig_link"/>
+  </joint>
+  <link name="right_sig_link">
+    <inertial>
+      <origin xyz="0 0 0" rpy="0 0 0"/>
+      <mass value="0.010"/>
+      <inertia ixx="0.0" ixy="0.0" ixz="0.0" iyy="0.0" iyz="0.0" izz="0.0"/>
+    </inertial>
+    <visual name='visual'>
+      <geometry>
+	    <box size="1 0.01 0.01"/>
+      </geometry>
+      <material name="black"/>
+    </visual>
+  </link>
+  <joint name="right_sig_joint" type="fixed">
+    <origin xyz="0.5 0 0" rpy="0 0 0"/>
+    <parent link="right_camera_link"/>
+    <child link="right_sig_link"/>
+  </joint>
   <transmission name="head_yaw_joint_tran">
     <type>transmission_interface/SimpleTransmission</type>

Commit message: Texture added

File: src/heads/urdf/head.xacro (robot description, xacro)
@@ -66,5 +66,5 @@
      <origin xyz="0 -1.5 0" rpy="0 0 0" />
       <geometry>
-        <mesh filename="package://heads/models/head.dae"/>
+        <mesh filename="package://heads/models/head/head.dae"/>
       </geometry>
     </collision>
@@ -72,5 +72,5 @@
      <origin xyz="0 -1.5 0" rpy="0 0 0" />
       <geometry>
-        <mesh filename="package://heads/models/head.dae"/>
+        <mesh filename="package://heads/models/head/head.dae"/>
       </geometry>
       <material name="orange"/>

Commit message: merged

File: src/heads/urdf/head.xacro (robot description, xacro)
@@ -15,10 +15,10 @@
     <collision name='collision'>
       <geometry>
-        <mesh filename="package://heads/models/torso.dae"/>
+        <mesh filename="package://heads/models/new_model2/torso.dae"/>
       </geometry>
     </collision>
     <visual name='visual'>
       <geometry>
-        <mesh filename="package://heads/models/torso.dae"/>
+        <mesh filename="package://heads/models/new_model2/torso.dae"/>
       </geometry>
       <material name="black"/>
@@ -66,5 +66,5 @@
      <origin xyz="0 -1.5 0" rpy="0 0 0" />
       <geometry>
-        <mesh filename="package://heads/models/head/head.dae"/>
+        <mesh filename="package://heads/models/new_model2/head/head.dae"/>
       </geometry>
     </collision>
@@ -72,5 +72,5 @@
      <origin xyz="0 -1.5 0" rpy="0 0 0" />
       <geometry>
-        <mesh filename="package://heads/models/head/head.dae"/>
+        <mesh filename="package://heads/models/new_model2/head/head.dae"/>
       </geometry>
       <material name="orange"/>
@@ -232,4 +232,5 @@
     <child link="left_camera_link"/>
   </joint>
+<!--
   <link name="left_sig_link">
     <inertial>
@@ -250,4 +251,6 @@
     <child link="left_sig_link"/>
   </joint>
+  -->
+  <!--
   <link name="right_sig_link">
     <inertial>
@@ -268,4 +271,5 @@
     <child link="right_sig_link"/>
   </joint>
+  -->
   <transmission name="head_yaw_joint_tran">
     <type>transmission_interface/SimpleTransmission</type>
